Commit message: update

File: control_robotarm/cybathlon_robotarm.URDF (robot description, URDF)
Before this commit: robot test_robot, 5 links, 4 joints
Joints:
- joint joint0: origin xyz=0 0 0 rpy=0 0 0 -> xyz=0 0 0 rpy=0 -0.3491 0
- joint joint1: axis 1 0 0 -> -1 0 0; origin xyz=0 0 0.075 rpy=0 0 0 -> xyz=0 0 0.075 rpy=-0.3491 0 0
- joint joint2: origin xyz=0.045 0 0.802 rpy=0 0 0 -> xyz=0.045 0 0.802 rpy=0 0.6981 0
